File: hw/c1-encoder-review/aux2.kicad_sch (KiCad schematic)
At the start: 9 parts, among them J2 0512810898, J3 BATTERY 2.7-3.6V, U7 THVD2442DRCR

Commit message: Add TI transceiver footprint and conditional loaded power budget
Parts:
- U7: footprint (none) -> Encoder:TI_DRC0010J
